File: pcb/pmm.brd (EAGLE design)
At the start: 81.6 x 43 mm, 34 parts, among them IC3 STM32F042F4, J1 AUDIO_JACK_3.5MM_PTH, J2 FFC3B07-05-T, SW3 324_SW, SW4 324_SW, U2 USBC_16P, U4 XC6206_DEV

Commit message: working on PCB
Parts:
- removed JP2, JP3: (no value), pinhead:1X02
- added C3: 1uF, clock:0805
- added R3, R6: 5.1K, joyAnalog:0805
- added U$8, U$9: PINHD1X2, adafruit_changed:1X02
- C2: value 1uF -> 100nF
- C4: value 1uF -> 2.2uF
- R4: value 1K -> 5K1
- moved U4 16.2 mm to (34.0, -22.9), turned to 270 degrees
- moved R4 13.0 mm to (35.3, -11.4)
- moved LED1 12.6 mm to (35.3, -9.69)
- moved C1 9.04 mm to (34.2, -19.9)
- moved R1 1.61 mm to (35.3, -5.08)
- moved R2 1.61 mm to (35.3, -7.87)
Connections:
- new net N$1: BT1.+, JP1.1
- new net PC_SYNC: IC3.10, J1.TIP, R6.1, U$8.2
- new net USER_LED: IC3.9, LED1.A
- net +3V3: now also JP1.2, R3.1, R6.2, U$6.1; no longer JP1.3, LED1.A, U4.2
- net GND: now also C3.1, J1.SLEEVE, R4.1, U$8.1, U$9.2
- net LIGHT_SENSE: now also IC3.2, U$9.1
- net N$2: now also R3.2
- net N$3: now also C3.2, JP1.3, U4.2; no longer BT1.+, JP1.2
- net OLED_CS: now also IC3.3
- net OLED_DC: now also IC3.7
- net OLED_RESET: now also IC3.6
Routing:
- net LIGHT_SENSE: track 0.00 -> 67.4 mm
- net OLED_DC: track 0.00 -> 61.3 mm, vias 0 -> 2
- net OLED_RESET: track 7.50 -> 66.7 mm, vias 0 -> 2
- net OLED_CS: track 0.00 -> 56.1 mm, vias 0 -> 2
- net +3V3: track 111.5 -> 134.5 mm, vias 7 -> 6
- net +5V: track 16.0 -> 35.3 mm
- net PC_SYNC: track 0.00 -> 13.2 mm
- net N$3: track 13.2 -> 25.6 mm
- net N$1: track 0.00 -> 9.71 mm
- net USER_LED: track 0.00 -> 7.99 mm
- net N$5: track 0.00 -> 1.81 mm
- net BUTTON2: track 42.2 -> 43.9 mm
- net N$2: track 44.4 -> 43.4 mm
- net GND: track 12.7 -> 11.8 mm, vias 0 -> 5
Other:
- outline, holes or cut-outs redrawn
- board text added: "DFU"
- board text added: "OFF"
- board text added: "ON"
- board text added: "RESET"
- board text removed: "middle pin on 3v3, left pin coin battery, right pin regulator output move regulator down twoards the edge"

Commit message: working on PCB
Parts:
- U$3, U$4, U$5: value POGO_1.5MM_HOLE -> POGO_TH001; device apricot:POGO_1.5 -> apricot:POGO_1.8
- moved U$9 2.54 mm to (-15.6, -23.4)
Connections:
- net N$1 renamed VBAT
Routing:
- net +3V3: track 134.5 -> 136.9 mm
- net LIGHT_SENSE: track 67.4 -> 68.9 mm
Other:
- board text added: "LS"
- board text added: "PC"
Changed lines of the file:
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@@
 <text x="2.4642" y="-17.4176" size="2.1844" layer="25" align="center">ON</text>
 <text x="9.3222" y="-17.4176" size="2.1844" layer="25" align="center">OFF</text>
+<rectangle x1="-7.239" y1="-17.272" x2="1.143" y2="-9.906" layer="16"/>
+<text x="32.893" y="-13.335" size="1.27" layer="25" align="center">PC</text>
+<text x="32.893" y="-15.875" size="1.27" layer="25" rot="R180" align="center">G</text>
+<text x="-16.891" y="-20.828" size="1.27" layer="25" rot="R90" align="center">LS</text>
+<text x="-14.3696" y="-20.4982" size="1.27" layer="25" rot="R270" align="center">GND</text>
 </plain>
 <attributes>
@@
 </element>
 <element name="R5" library="joyAnalog" package="0805" value="5.1K" x="-11.1286" y="-20" smashed="yes" rot="R270">
-<attribute name="NAME" x="-11.9071" y="-19.9784" size="0.8128" layer="25" rot="R90"/>
+<attribute name="NAME" x="-12.1611" y="-20.4864" size="0.8128" layer="25" rot="R90"/>
 </element>
 <element name="U4" library="3pos_slide_switch" package="SOT23R_INFINEON" value="XC6206_DEV" x="34.036" y="-22.86" smashed="yes" rot="R270"/>
@@
 <element name="U$1" library="3pos_slide_switch_centered" package="M2_SCREW_FOOT" value="M2_SCREW_DEV" x="10.3" y="3.5" locked="yes" smashed="yes"/>
 <element name="U$2" library="3pos_slide_switch_centered" package="M2_SCREW_FOOT" value="M2_SCREW_DEV" x="2.3" y="3.5" locked="yes" smashed="yes"/>
-<element name="U$3" library="apricot" package="POGO_1.5" value="POGO_1.5MM_HOLE" x="6.3" y="9.5" locked="yes" smashed="yes"/>
-<element name="U$4" library="apricot" package="POGO_1.5" value="POGO_1.5MM_HOLE" x="2.05" y="14" locked="yes" smashed="yes"/>
-<element name="U$5" library="apricot" package="POGO_1.5" value="POGO_1.5MM_HOLE" x="10.55" y="14" locked="yes" smashed="yes"/>
+<element name="U$3" library="apricot" package="POGO_1.8" value="POGO_TH001" x="6.3" y="9.5" locked="yes" smashed="yes"/>
+<element name="U$4" library="apricot" package="POGO_1.8" value="POGO_TH001" x="2.05" y="14" locked="yes" smashed="yes"/>
+<element name="U$5" library="apricot" package="POGO_1.8" value="POGO_TH001" x="10.55" y="14" locked="yes" smashed="yes"/>
 <element name="U1" library="lul" package="LUL_UG-2864HSWEG01_1.3_WRAPAROUND" value="" x="-24.384" y="-9.525" smashed="yes" rot="R90"/>
 <element name="R7" library="SparkFun-Passives" package="0805" value="390K" x="-27.559" y="-11.049" smashed="yes">
@@
 </element>
 <element name="U$8" library="adafruit_changed" package="1X02" value="PINHD1X2" x="34.671" y="-14.605" smashed="yes" rot="R90"/>
-<element name="U$9" library="adafruit_changed" package="1X02" value="PINHD1X2" x="-18.161" y="-23.368" smashed="yes"/>
+<element name="U$9" library="adafruit_changed" package="1X02" value="PINHD1X2" x="-15.621" y="-23.368" smashed="yes"/>
 <element name="C3" library="clock" package="0805" value="1uF" x="30.861" y="-22.86" smashed="yes" rot="R270">
 <attribute name="NAME" x="29.0195" y="-22.352" size="0.8128" layer="25" rot="R270"/>
@@
 <wire x1="-3.6" y1="-18.875" x2="-5.794" y2="-18.875" width="0.508" layer="1"/>
 <wire x1="-5.794" y1="-18.875" x2="-5.842" y2="-18.923" width="0.508" layer="1"/>
-<wire x1="-28.829" y1="-20.066" x2="-28.829" y2="-10.795" width="0.508" layer="16"/>
-<wire x1="-28.829" y1="-10.795" x2="-30.48" y2="-9.144" width="0.508" layer="16"/>
 <contactref element="JP1" pad="2"/>
 <contactref element="C2" pad="2"/>
@@
 <wire x1="28.25" y1="-9.088" x2="28.967" y2="-8.371" width="0.2032" layer="1"/>
 <wire x1="28.967" y1="-8.371" x2="28.967" y2="-7.874" width="0.2032" layer="1"/>
+<wire x1="-30.48" y1="-9.144" x2="-27.813" y2="-9.144" width="0.508" layer="16"/>
+<wire x1="-26.797" y1="-10.16" x2="-26.797" y2="-20.066" width="0.508" layer="16"/>
+<wire x1="-27.813" y1="-9.144" x2="-26.797" y2="-10.16" width="0.508" layer="16"/>
 </signal>
 <signal name="USB_DP">
@@
 <wire x1="24.765" y1="-20.066" x2="11.557" y2="-20.066" width="0.1524" layer="1"/>
 <wire x1="10.287" y1="-18.796" x2="8.255" y2="-18.796" width="0.1524" layer="1"/>
-<wire x1="1.057" y1="-21.971" x2="0.211" y2="-21.125" width="0.1524" layer="1"/>
-<wire x1="1.057" y1="-21.971" x2="6.985" y2="-21.971" width="0.1524" layer="1"/>
-<wire x1="8.255" y1="-18.796" x2="7.7724" y2="-19.2786" width="0.1524" layer="1"/>
-<wire x1="7.7724" y1="-21.1836" x2="6.985" y2="-21.971" width="0.1524" layer="1"/>
-<wire x1="7.7724" y1="-19.2786" x2="7.7724" y2="-21.1836" width="0.1524" layer="1"/>
+<wire x1="1.1332" y1="-22.0472" x2="0.211" y2="-21.125" width="0.1524" layer="1"/>
+<wire x1="1.1332" y1="-22.0472" x2="7.2898" y2="-22.0472" width="0.1524" layer="1"/>
+<wire x1="8.255" y1="-18.796" x2="7.747" y2="-19.304" width="0.1524" layer="1"/>
+<wire x1="7.747" y1="-21.59" x2="7.2898" y2="-22.0472" width="0.1524" layer="1"/>
+<wire x1="7.747" y1="-19.304" x2="7.747" y2="-21.59" width="0.1524" layer="1"/>
 </signal>
 <signal name="N$5">
@@
 <contactref element="U$9" pad="1"/>
 <wire x1="-27.813" y1="-18.251" x2="-27.813" y2="-21.844" width="0.2032" layer="1"/>
-<wire x1="-26.289" y1="-23.368" x2="-19.431" y2="-23.368" width="0.2032" layer="1"/>
+<wire x1="-26.289" y1="-23.368" x2="-16.891" y2="-23.368" width="0.2032" layer="1"/>
 <wire x1="-27.813" y1="-21.844" x2="-26.289" y2="-23.368" width="0.2032" layer="1"/>
-<wire x1="-19.431" y1="-23.368" x2="-13.589" y2="-17.526" width="0.1524" layer="1"/>
-<wire x1="-13.589" y1="-17.526" x2="-1.143" y2="-17.526" width="0.1524" layer="1"/>
-<wire x1="-1.143" y1="-17.526" x2="2.794" y2="-21.463" width="0.1524" layer="1"/>
-<wire x1="2.794" y1="-21.463" x2="6.858" y2="-21.463" width="0.1524" layer="1"/>
+<wire x1="-16.891" y1="-23.368" x2="-16.891" y2="-21.336" width="0.1524" layer="1"/>
+<wire x1="-13.208" y1="-17.653" x2="-16.891" y2="-21.336" width="0.1524" layer="1"/>
+<wire x1="-13.208" y1="-17.653" x2="-1.016" y2="-17.653" width="0.1524" layer="1"/>
+<wire x1="-1.016" y1="-17.653" x2="2.9972" y2="-21.6662" width="0.1524" layer="1"/>
+<wire x1="2.9972" y1="-21.6662" x2="7.0358" y2="-21.6662" width="0.1524" layer="1"/>
 <wire x1="10.668" y1="-14.986" x2="26.162" y2="-14.986" width="0.1524" layer="1"/>
-<wire x1="6.858" y1="-21.463" x2="7.3914" y2="-20.9296" width="0.1524" layer="1"/>
-<wire x1="7.3914" y1="-20.9296" x2="7.3914" y2="-18.2626" width="0.1524" layer="1"/>
+<wire x1="7.0358" y1="-21.6662" x2="7.3914" y2="-21.3106" width="0.1524" layer="1"/>
+<wire x1="7.3914" y1="-21.3106" x2="7.3914" y2="-18.2626" width="0.1524" layer="1"/>
 <wire x1="7.3914" y1="-18.2626" x2="10.668" y2="-14.986" width="0.1524" layer="1"/>
 <contactref element="IC3" pad="2"/>
@@
 <wire x1="26.3" y1="-15.124" x2="26.3" y2="-15.8718" width="0.1524" layer="1"/>
 </signal>
-<signal name="N$1">
+<signal name="VBAT">
 <contactref element="BT1" pad="+"/>
 <contactref element="JP1" pad="1"/>
