File: pcb/pmm.brd (EAGLE design)
At the start: 78.6 x 43 mm, 43 parts, among them IC3 STM32F042F4, J1 AUDIO_JACK_3.5MM_PTH, J2 FFC3B07-05-T, SW3 324_SW, SW4 324_SW, U2 USBC_16P, U4 XC6206_DEV

Commit message: updated PCB
Parts:
- removed U$11, U$13, U$14, U$5, U$9: SPRING_CONTACT, apricot:SPRING_CONTACT
- added U$3: HOTSHOE, apricot:HOTSHOE_RAIL
- U$4: value SPRING_CONTACT -> HOTSHOE; device apricot:SPRING_CONTACT -> apricot:HOTSHOE_RAIL
- moved U$4 5.83 mm to (12.4, 9.65)
- moved U$15 1.55 mm to (0.07, 9.61)
- moved U$10 1.55 mm to (12.5, 9.61)
- moved BT1 1.27 mm to (-14.6, -14.8)
Connections:
- net GND: now also U$3.P$1; no longer U$11.P$1, U$13.P$1, U$14.P$1, U$5.P$1, U$9.P$1
Routing:
- net VBAT: track 8.47 -> 7.20 mm
Other:
- board text added: "1.2mm Thick ENIG gold finish FDX0039B2 Spring contact"
Changed lines of the file:
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@@
 <setting verticaltext="up"/>
 </settings>
-<grid distance="5" unitdist="mil" unit="mil" style="lines" multiple="1" display="no" altdistance="1" altunitdist="mil" altunit="mil"/>
+<grid distance="10" unitdist="mil" unit="mil" style="lines" multiple="1" display="no" altdistance="1" altunitdist="mil" altunit="mil"/>
 <layers>
 <layer number="1" name="Top" color="4" fill="1" visible="yes" active="yes"/>
@@
 <text x="1.8292" y="-17.7986" size="2.1844" layer="25" align="center">ON</text>
 <text x="10.4652" y="-17.7986" size="2.1844" layer="25" align="center">OFF</text>
-<rectangle x1="-4.064" y1="-16.891" x2="4.318" y2="-9.525" layer="16"/>
+<rectangle x1="-4.064" y1="-17.907" x2="4.318" y2="-10.541" layer="16"/>
 <text x="32.639" y="-13.208" size="1.27" layer="25" rot="R90" align="center">PC</text>
 <text x="32.639" y="-15.875" size="1.27" layer="25" align="center">G</text>
@@
 <text x="-12.1408" y="-22.0376" size="1.27" layer="25" align="center">G</text>
 <text x="-14.6808" y="-22.0376" size="1.27" layer="25" align="center">V</text>
-<text x="-8.2038" y="-3.7016" size="2.1082" layer="25" align="center">PulseHPT.com</text>
+<text x="-6.9338" y="-3.4476" size="1.9304" layer="25" align="center">PulseHPT.com</text>
 <text x="14.6562" y="-13.6076" size="2.1082" layer="26" rot="MR0" align="center">PulseHPT.com
 dekuNukem 2023</text>
 <wire x1="0" y1="20" x2="0" y2="-1" width="0.1016" layer="51"/>
 <wire x1="12.6" y1="19" x2="12.6" y2="-1" width="0.1016" layer="51"/>
+<text x="-20.6498" y="12.3004" size="1.9304" layer="25" align="center">1.2mm Thick
+ENIG gold finish
+FDX0039B2 Spring contact</text>
 </plain>
 <attributes>
@@
 <attribute name="NAME" x="-28.7655" y="-7.62" size="0.8128" layer="25" rot="R90"/>
 </element>
-<element name="BT1" library="BU2032SM-G" package="BAT_BU2032SM-G" value="BU2032SM-G" x="-14.6" y="-13.5" smashed="yes" rot="MR0">
-<attribute name="AVAILABILITY" value="In Stock" x="-14.6" y="-13.5" size="1.778" layer="28" rot="MR0" display="off"/>
-<attribute name="CHECK_PRICES" value="https://www.snapeda.com/parts/BU2032SM-G/Memory+Protection+Devices/view-part/?ref=eda" x="-14.6" y="-13.5" size="1.778" layer="28" rot="MR0" display="off"/>
-<attribute name="DESCRIPTION" value=" BATTERY HOLDER COIN 20MM SMD " x="-14.6" y="-13.5" size="1.778" layer="28" rot="MR0" display="off"/>
-<attribute name="MF" value="MPD" x="-14.6" y="-13.5" size="1.778" layer="28" rot="MR0" display="off"/>
-<attribute name="MP" value="BU2032SM-G" x="-14.6" y="-13.5" size="1.778" layer="28" rot="MR0" display="off"/>
-<attribute name="PACKAGE" value="None" x="-14.6" y="-13.5" size="1.778" layer="28" rot="MR0" display="off"/>
-<attribute name="PRICE" value="None" x="-14.6" y="-13.5" size="1.778" layer="28" rot="MR0" display="off"/>
-<attribute name="PURCHASE-URL" value="https://www.snapeda.com/api/url_track_click_mouser/?unipart_id=4219599&amp;manufacturer=MPD&amp;part_name=BU2032SM-G&amp;search_term=battery holder" x="-14.6" y="-13.5" size="1.778" layer="28" rot="MR0" display="off"/>
-<attribute name="SNAPEDA_LINK" value="https://www.snapeda.com/parts/BU2032SM-G/Memory+Protection+Devices/view-part/?ref=snap" x="-14.6" y="-13.5" size="1.778" layer="28" rot="MR0" display="off"/>
+<element name="BT1" library="BU2032SM-G" package="BAT_BU2032SM-G" value="BU2032SM-G" x="-14.6" y="-14.77" smashed="yes" rot="MR0">
+<attribute name="AVAILABILITY" value="In Stock" x="-14.6" y="-14.77" size="1.778" layer="28" rot="MR0" display="off"/>
+<attribute name="CHECK_PRICES" value="https://www.snapeda.com/parts/BU2032SM-G/Memory+Protection+Devices/view-part/?ref=eda" x="-14.6" y="-14.77" size="1.778" layer="28" rot="MR0" display="off"/>
+<attribute name="DESCRIPTION" value=" BATTERY HOLDER COIN 20MM SMD " x="-14.6" y="-14.77" size="1.778" layer="28" rot="MR0" display="off"/>
+<attribute name="MF" value="MPD" x="-14.6" y="-14.77" size="1.778" layer="28" rot="MR0" display="off"/>
+<attribute name="MP" value="BU2032SM-G" x="-14.6" y="-14.77" size="1.778" layer="28" rot="MR0" display="off"/>
+<attribute name="PACKAGE" value="None" x="-14.6" y="-14.77" size="1.778" layer="28" rot="MR0" display="off"/>
+<attribute name="PRICE" value="None" x="-14.6" y="-14.77" size="1.778" layer="28" rot="MR0" display="off"/>
+<attribute name="PURCHASE-URL" value="https://www.snapeda.com/api/url_track_click_mouser/?unipart_id=4219599&amp;manufacturer=MPD&amp;part_name=BU2032SM-G&amp;search_term=battery holder" x="-14.6" y="-14.77" size="1.778" layer="28" rot="MR0" display="off"/>
+<attribute name="SNAPEDA_LINK" value="https://www.snapeda.com/parts/BU2032SM-G/Memory+Protection+Devices/view-part/?ref=snap" x="-14.6" y="-14.77" size="1.778" layer="28" rot="MR0" display="off"/>
 </element>
 <element name="J1" library="SparkFun-Connectors" package="AUDIO-JACK" value="AUDIO_JACK_3.5MM_PTH" x="43.688" y="-18.669" smashed="yes" rot="R180">
@@
 <attribute name="NAME" x="-13.208" y="-16.7005" size="0.8128" layer="25" rot="R180"/>
 </element>
-<element name="U$11" library="apricot" package="SPRING_CONTACT" value="SPRING_CONTACT" x="-1.524" y="3.556" smashed="yes"/>
-<element name="U$13" library="apricot" package="SPRING_CONTACT" value="SPRING_CONTACT" x="-1.524" y="9.398" smashed="yes"/>
-<element name="U$14" library="apricot" package="SPRING_CONTACT" value="SPRING_CONTACT" x="-1.524" y="15.24" smashed="yes"/>
-<element name="U$4" library="apricot" package="SPRING_CONTACT" value="SPRING_CONTACT" x="14.097" y="15.24" smashed="yes"/>
-<element name="U$5" library="apricot" package="SPRING_CONTACT" value="SPRING_CONTACT" x="14.097" y="9.398" smashed="yes"/>
-<element name="U$9" library="apricot" package="SPRING_CONTACT" value="SPRING_CONTACT" x="14.097" y="3.556" smashed="yes"/>
-<element name="U$10" library="apricot" package="HOTSHOE_RAIL" value="HOTSHOE" x="13.975" y="9.354" smashed="yes" rot="MR0"/>
-<element name="U$15" library="apricot" package="HOTSHOE_RAIL" value="HOTSHOE" x="-1.455" y="9.354" smashed="yes" rot="MR0"/>
+<element name="U$10" library="apricot" package="HOTSHOE_RAIL" value="HOTSHOE" x="12.451" y="9.608" smashed="yes" rot="MR0"/>
+<element name="U$15" library="apricot" package="HOTSHOE_RAIL" value="HOTSHOE" x="0.069" y="9.608" smashed="yes" rot="MR0"/>
 <element name="U$2" library="apricot" package="SPRING_CONTACT" value="SPRING_CONTACT" x="6.3" y="10.3" smashed="yes" rot="MR0"/>
+<element name="U$3" library="apricot" package="HOTSHOE_RAIL" value="HOTSHOE" x="0" y="9.652" smashed="yes"/>
+<element name="U$4" library="apricot" package="HOTSHOE_RAIL" value="HOTSHOE" x="12.446" y="9.652" smashed="yes"/>
 </elements>
 <signals>
@@
 <contactref element="R9" pad="2"/>
 <via x="-0.381" y="-23.495" extent="1-16" drill="0.5"/>
-<contactref element="U$13" pad="P$1"/>
-<contactref element="U$11" pad="P$1"/>
-<contactref element="U$14" pad="P$1"/>
-<contactref element="U$5" pad="P$1"/>
-<contactref element="U$9" pad="P$1"/>
-<contactref element="U$4" pad="P$1"/>
 <contactref element="U$10" pad="P$1"/>
 <contactref element="U$15" pad="P$1"/>
 <via x="18.415" y="-17.272" extent="1-16" drill="0.5"/>
+<contactref element="U$3" pad="P$1"/>
+<contactref element="U$4" pad="P$1"/>
 </signal>
 <signal name="+3V3">
@@
 <contactref element="BT1" pad="+"/>
 <contactref element="JP1" pad="1"/>
-<wire x1="-0.1" y1="-13.5" x2="3.76" y2="-17.36" width="0.508" layer="16"/>
-<wire x1="3.76" y1="-17.36" x2="3.76" y2="-20.373" width="0.508" layer="16"/>
+<wire x1="-0.1" y1="-14.77" x2="3.76" y2="-18.63" width="0.508" layer="16"/>
+<wire x1="3.76" y1="-18.63" x2="3.76" y2="-20.373" width="0.508" layer="16"/>
 </signal>
 <signal name="N$3">

Commit message: adjusted PCB
Parts:
- C2: value 100nF -> 2.2uF
- R4: value 5K1 -> 2K
- moved U$10 1.02 mm to (13.5, 9.61)
- moved U$15 1.02 mm to (-0.95, 9.61)
- moved U$3 1.02 mm to (-1.02, 9.65)
- moved U$4 1.02 mm to (13.5, 9.65)
- moved JP2 0.13 mm to (-12.2, -23.9)
- moved BT1 0.13 mm to (-14.6, -14.6)
Changed lines of the file:
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@@
 <setting verticaltext="up"/>
 </settings>
-<grid distance="10" unitdist="mil" unit="mil" style="lines" multiple="1" display="no" altdistance="1" altunitdist="mil" altunit="mil"/>
+<grid distance="20" unitdist="mil" unit="mil" style="lines" multiple="1" display="no" altdistance="1" altunitdist="mil" altunit="mil"/>
 <layers>
 <layer number="1" name="Top" color="4" fill="1" visible="yes" active="yes"/>
@@
 <attribute name="VALUE" x="34.061" y="-12.228" size="1.27" layer="27"/>
 </element>
-<element name="R4" library="SparkFun-Passives" package="0805" value="5K1" x="35.331" y="-11.434" smashed="yes">
+<element name="R4" library="SparkFun-Passives" package="0805" value="2K" x="35.331" y="-11.434" smashed="yes">
 <attribute name="NAME" x="37.0074" y="-11.7769" size="0.8128" layer="25"/>
 </element>
@@
 </element>
 <element name="U4" library="3pos_slide_switch" package="SOT23R_INFINEON" value="XC6206_DEV" x="34.036" y="-22.86" smashed="yes" rot="R270"/>
-<element name="C2" library="clock" package="0805" value="100nF" x="28.067" y="-7.874" smashed="yes">
+<element name="C2" library="clock" package="0805" value="2.2uF" x="28.067" y="-7.874" smashed="yes">
 <attribute name="NAME" x="30.7378" y="-7.4765" size="0.8128" layer="25" rot="R180"/>
 </element>
@@
 <attribute name="NAME" x="-28.7655" y="-7.62" size="0.8128" layer="25" rot="R90"/>
 </element>
-<element name="BT1" library="BU2032SM-G" package="BAT_BU2032SM-G" value="BU2032SM-G" x="-14.6" y="-14.77" smashed="yes" rot="MR0">
-<attribute name="AVAILABILITY" value="In Stock" x="-14.6" y="-14.77" size="1.778" layer="28" rot="MR0" display="off"/>
-<attribute name="CHECK_PRICES" value="https://www.snapeda.com/parts/BU2032SM-G/Memory+Protection+Devices/view-part/?ref=eda" x="-14.6" y="-14.77" size="1.778" layer="28" rot="MR0" display="off"/>
-<attribute name="DESCRIPTION" value=" BATTERY HOLDER COIN 20MM SMD " x="-14.6" y="-14.77" size="1.778" layer="28" rot="MR0" display="off"/>
-<attribute name="MF" value="MPD" x="-14.6" y="-14.77" size="1.778" layer="28" rot="MR0" display="off"/>
-<attribute name="MP" value="BU2032SM-G" x="-14.6" y="-14.77" size="1.778" layer="28" rot="MR0" display="off"/>
-<attribute name="PACKAGE" value="None" x="-14.6" y="-14.77" size="1.778" layer="28" rot="MR0" display="off"/>
-<attribute name="PRICE" value="None" x="-14.6" y="-14.77" size="1.778" layer="28" rot="MR0" display="off"/>
-<attribute name="PURCHASE-URL" value="https://www.snapeda.com/api/url_track_click_mouser/?unipart_id=4219599&amp;manufacturer=MPD&amp;part_name=BU2032SM-G&amp;search_term=battery holder" x="-14.6" y="-14.77" size="1.778" layer="28" rot="MR0" display="off"/>
-<attribute name="SNAPEDA_LINK" value="https://www.snapeda.com/parts/BU2032SM-G/Memory+Protection+Devices/view-part/?ref=snap" x="-14.6" y="-14.77" size="1.778" layer="28" rot="MR0" display="off"/>
+<element name="BT1" library="BU2032SM-G" package="BAT_BU2032SM-G" value="BU2032SM-G" x="-14.6" y="-14.643" smashed="yes" rot="MR0">
+<attribute name="AVAILABILITY" value="In Stock" x="-14.6" y="-14.643" size="1.778" layer="28" rot="MR0" display="off"/>
+<attribute name="CHECK_PRICES" value="https://www.snapeda.com/parts/BU2032SM-G/Memory+Protection+Devices/view-part/?ref=eda" x="-14.6" y="-14.643" size="1.778" layer="28" rot="MR0" display="off"/>
+<attribute name="DESCRIPTION" value=" BATTERY HOLDER COIN 20MM SMD " x="-14.6" y="-14.643" size="1.778" layer="28" rot="MR0" display="off"/>
+<attribute name="MF" value="MPD" x="-14.6" y="-14.643" size="1.778" layer="28" rot="MR0" display="off"/>
+<attribute name="MP" value="BU2032SM-G" x="-14.6" y="-14.643" size="1.778" layer="28" rot="MR0" display="off"/>
+<attribute name="PACKAGE" value="None" x="-14.6" y="-14.643" size="1.778" layer="28" rot="MR0" display="off"/>
+<attribute name="PRICE" value="None" x="-14.6" y="-14.643" size="1.778" layer="28" rot="MR0" display="off"/>
+<attribute name="PURCHASE-URL" value="https://www.snapeda.com/api/url_track_click_mouser/?unipart_id=4219599&amp;manufacturer=MPD&amp;part_name=BU2032SM-G&amp;search_term=battery holder" x="-14.6" y="-14.643" size="1.778" layer="28" rot="MR0" display="off"/>
+<attribute name="SNAPEDA_LINK" value="https://www.snapeda.com/parts/BU2032SM-G/Memory+Protection+Devices/view-part/?ref=snap" x="-14.6" y="-14.643" size="1.778" layer="28" rot="MR0" display="off"/>
 </element>
 <element name="J1" library="SparkFun-Connectors" package="AUDIO-JACK" value="AUDIO_JACK_3.5MM_PTH" x="43.688" y="-18.669" smashed="yes" rot="R180">
@@
 <attribute name="NAME" x="29.0195" y="-21.971" size="0.8128" layer="25" rot="R270"/>
 </element>
-<element name="JP2" library="adafruit_changed" package="1X03-CLEANBIG" value="" x="-12.192" y="-23.749" smashed="yes" rot="R180">
-<attribute name="VALUE" x="-8.382" y="-20.574" size="1.27" layer="27" rot="R180"/>
+<element name="JP2" library="adafruit_changed" package="1X03-CLEANBIG" value="" x="-12.192" y="-23.876" smashed="yes" rot="R180">
+<attribute name="VALUE" x="-8.382" y="-20.701" size="1.27" layer="27" rot="R180"/>
 </element>
 <element name="R9" library="joyAnalog" package="0805" value="270K" x="-13.843" y="-18.542" smashed="yes" rot="R180">
 <attribute name="NAME" x="-13.208" y="-16.7005" size="0.8128" layer="25" rot="R180"/>
 </element>
-<element name="U$10" library="apricot" package="HOTSHOE_RAIL" value="HOTSHOE" x="12.451" y="9.608" smashed="yes" rot="MR0"/>
-<element name="U$15" library="apricot" package="HOTSHOE_RAIL" value="HOTSHOE" x="0.069" y="9.608" smashed="yes" rot="MR0"/>
+<element name="U$10" library="apricot" package="HOTSHOE_RAIL" value="HOTSHOE" x="13.467" y="9.608" smashed="yes" rot="MR0"/>
+<element name="U$15" library="apricot" package="HOTSHOE_RAIL" value="HOTSHOE" x="-0.947" y="9.608" smashed="yes" rot="MR0"/>
 <element name="U$2" library="apricot" package="SPRING_CONTACT" value="SPRING_CONTACT" x="6.3" y="10.3" smashed="yes" rot="MR0"/>
-<element name="U$3" library="apricot" package="HOTSHOE_RAIL" value="HOTSHOE" x="0" y="9.652" smashed="yes"/>
-<element name="U$4" library="apricot" package="HOTSHOE_RAIL" value="HOTSHOE" x="12.446" y="9.652" smashed="yes"/>
+<element name="U$3" library="apricot" package="HOTSHOE_RAIL" value="HOTSHOE" x="-1.016" y="9.652" smashed="yes"/>
+<element name="U$4" library="apricot" package="HOTSHOE_RAIL" value="HOTSHOE" x="13.462" y="9.652" smashed="yes"/>
 </elements>
 <signals>
@@
 <contactref element="JP2" pad="3"/>
 <wire x1="-5.842" y1="-18.923" x2="-11.303" y2="-18.923" width="0.508" layer="16"/>
-<wire x1="-14.732" y1="-22.352" x2="-14.732" y2="-23.749" width="0.508" layer="16"/>
+<wire x1="-14.732" y1="-22.352" x2="-14.732" y2="-23.876" width="0.508" layer="16"/>
 <wire x1="-11.303" y1="-18.923" x2="-14.732" y2="-22.352" width="0.508" layer="16"/>
-<wire x1="-14.732" y1="-23.749" x2="-20.114" y2="-23.749" width="0.508" layer="16"/>
-<wire x1="-20.114" y1="-23.749" x2="-23.797" y2="-20.066" width="0.508" layer="16"/>
+<wire x1="-14.732" y1="-23.876" x2="-19.987" y2="-23.876" width="0.508" layer="16"/>
+<wire x1="-19.987" y1="-23.876" x2="-23.797" y2="-20.066" width="0.508" layer="16"/>
 </signal>
 <signal name="USB_DP">
@@
 <signal name="LIGHT_SENSE">
 <contactref element="J2" pad="3"/>
-<wire x1="-1.27" y1="-17.399" x2="2.9972" y2="-21.6662" width="0.1524" layer="1"/>
-<wire x1="2.9972" y1="-21.6662" x2="7.0358" y2="-21.6662" width="0.1524" layer="1"/>
+<wire x1="-1.778" y1="-17.399" x2="2.4892" y2="-21.6662" width="0.1524" layer="1"/>
+<wire x1="2.4892" y1="-21.6662" x2="7.0358" y2="-21.6662" width="0.1524" layer="1"/>
 <wire x1="10.795" y1="-14.859" x2="26.162" y2="-14.859" width="0.1524" layer="1"/>
 <wire x1="7.0358" y1="-21.6662" x2="7.3914" y2="-21.3106" width="0.1524" layer="1"/>
@@
 <contactref element="JP2" pad="1"/>
 <contactref element="R9" pad="1"/>
-<wire x1="-1.27" y1="-17.399" x2="-12.954" y2="-17.399" width="0.2032" layer="1"/>
-<wire x1="-12.954" y1="-17.399" x2="-14.732" y2="-17.399" width="0.2032" layer="1"/>
-<wire x1="-14.732" y1="-17.399" x2="-21.336" y2="-17.399" width="0.2032" layer="1"/>
+<wire x1="-1.778" y1="-17.399" x2="-12.954" y2="-17.399" width="0.2032" layer="1"/>
+<wire x1="-12.954" y1="-17.399" x2="-21.336" y2="-17.399" width="0.2032" layer="1"/>
 <wire x1="-24.813" y1="-18.251" x2="-24.813" y2="-16.812" width="0.2032" layer="1"/>
 <wire x1="-24.813" y1="-16.812" x2="-24.511" y2="-16.51" width="0.2032" layer="1"/>
 <wire x1="-24.511" y1="-16.51" x2="-22.225" y2="-16.51" width="0.2032" layer="1"/>
 <wire x1="-22.225" y1="-16.51" x2="-21.336" y2="-17.399" width="0.2032" layer="1"/>
-<wire x1="-14.743" y1="-17.41" x2="-14.732" y2="-17.399" width="0.2032" layer="1"/>
-<wire x1="-12.943" y1="-20.458" x2="-12.943" y2="-18.542" width="0.2032" layer="1"/>
-<wire x1="-9.652" y1="-23.749" x2="-12.943" y2="-20.458" width="0.2032" layer="1"/>
+<wire x1="-12.943" y1="-20.585" x2="-12.943" y2="-18.542" width="0.2032" layer="1"/>
+<wire x1="-9.652" y1="-23.876" x2="-12.943" y2="-20.585" width="0.2032" layer="1"/>
 <wire x1="-12.943" y1="-18.542" x2="-12.954" y2="-18.531" width="0.2032" layer="1"/>
 <wire x1="-12.954" y1="-18.531" x2="-12.954" y2="-17.399" width="0.2032" layer="1"/>
@@
 <contactref element="BT1" pad="+"/>
 <contactref element="JP1" pad="1"/>
-<wire x1="-0.1" y1="-14.77" x2="3.76" y2="-18.63" width="0.508" layer="16"/>
-<wire x1="3.76" y1="-18.63" x2="3.76" y2="-20.373" width="0.508" layer="16"/>
+<wire x1="-0.1" y1="-14.643" x2="3.76" y2="-18.503" width="0.508" layer="16"/>
+<wire x1="3.76" y1="-18.503" x2="3.76" y2="-20.373" width="0.508" layer="16"/>
 </signal>
 <signal name="N$3">

Commit message: cleaning up pcb
Parts:
- added U$14, U$16, U$5, U$9: HOTSHOE, apricot:HOTSHOE_RAIL
- C2, C23: value 2.2uF -> 1uF
- C3: value 1uF -> 2.2uF
- R4: value 2K -> 5.1K
- moved C3 25.4 mm to (5.97, -17.7), turned to 0 degrees
- moved JP2 20.9 mm to (-10.5, -3.07)
- moved U$10 5.12 mm to (14.1, 14.7)
- moved U$4 5.12 mm to (14.1, 14.7)
- moved U$15 5.11 mm to (-1.46, 14.7)
- moved U$3 5.09 mm to (-1.40, 14.7)
- turned R5 to 90 degrees
- turned SW4 to 0 degrees
Connections:
- net +3V3: now also C3.2
- net GND: now also U$14.P$1, U$16.P$1, U$5.P$1, U$9.P$1
- net N$3: no longer C3.2
Routing:
- net +3V3: track 134.5 -> 146.1 mm
- net LIGHT_SENSE: track 68.2 -> 77.2 mm, vias 0 -> 1
- net USB_DP: track 35.4 -> 35.9 mm
Other:
- board text added: "PulseHPT .com"
- board text removed: "PulseHPT.com"
