File: pcb/pmm.brd (EAGLE design)
At the start: 78.6 x 43 mm, 43 parts, among them IC3 STM32F042F4, J1 AUDIO_JACK_3.5MM_PTH, J2 FFC3B07-05-T, SW3 324_SW, SW4 324_SW, U2 USBC_16P, U4 XC6206_DEV

Commit message: cleaning up pcb
Parts:
- U$10, U$15, U$5, U$9: value HOTSHOE -> HOTSHOE_NOPASTE; device apricot:HOTSHOE_RAIL -> apricot:HOTSHOE_RAIL_NOPASTE
- moved U$2 0.25 mm to (6.30, 10.1)
Other:
- board text added: "LS"
- board text removed: "S"
Changed lines of the file:
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@@
 <grid distance="5" unitdist="mil" unit="mil" style="lines" multiple="1" display="no" altdistance="1" altunitdist="mil" altunit="mil"/>
 <layers>
-<layer number="1" name="Top" color="4" fill="1" visible="no" active="yes"/>
+<layer number="1" name="Top" color="4" fill="1" visible="yes" active="yes"/>
 <layer number="2" name="Route2" color="16" fill="1" visible="no" active="no"/>
 <layer number="3" name="Route3" color="17" fill="1" visible="no" active="no"/>
@@
 <layer number="19" name="Unrouted" color="6" fill="1" visible="yes" active="yes"/>
 <layer number="20" name="Dimension" color="24" fill="1" visible="yes" active="yes"/>
-<layer number="21" name="tPlace" color="7" fill="1" visible="no" active="yes"/>
-<layer number="22" name="bPlace" color="7" fill="1" visible="no" active="yes"/>
-<layer number="23" name="tOrigins" color="15" fill="1" visible="no" active="yes"/>
+<layer number="21" name="tPlace" color="7" fill="1" visible="yes" active="yes"/>
+<layer number="22" name="bPlace" color="7" fill="1" visible="yes" active="yes"/>
+<layer number="23" name="tOrigins" color="15" fill="1" visible="yes" active="yes"/>
 <layer number="24" name="bOrigins" color="15" fill="1" visible="yes" active="yes"/>
-<layer number="25" name="tNames" color="7" fill="1" visible="no" active="yes"/>
-<layer number="26" name="bNames" color="7" fill="1" visible="no" active="yes"/>
-<layer number="27" name="tValues" color="7" fill="1" visible="no" active="yes"/>
-<layer number="28" name="bValues" color="7" fill="1" visible="no" active="yes"/>
+<layer number="25" name="tNames" color="7" fill="1" visible="yes" active="yes"/>
+<layer number="26" name="bNames" color="7" fill="1" visible="yes" active="yes"/>
+<layer number="27" name="tValues" color="7" fill="1" visible="yes" active="yes"/>
+<layer number="28" name="bValues" color="7" fill="1" visible="yes" active="yes"/>
 <layer number="29" name="tStop" color="7" fill="3" visible="no" active="yes"/>
 <layer number="30" name="bStop" color="7" fill="6" visible="no" active="yes"/>
@@
 <layer number="37" name="tTest" color="7" fill="1" visible="no" active="yes"/>
 <layer number="38" name="bTest" color="7" fill="1" visible="no" active="yes"/>
-<layer number="39" name="tKeepout" color="4" fill="11" visible="no" active="yes"/>
+<layer number="39" name="tKeepout" color="4" fill="11" visible="yes" active="yes"/>
 <layer number="40" name="bKeepout" color="1" fill="11" visible="yes" active="yes"/>
-<layer number="41" name="tRestrict" color="4" fill="10" visible="no" active="yes"/>
+<layer number="41" name="tRestrict" color="4" fill="10" visible="yes" active="yes"/>
 <layer number="42" name="bRestrict" color="1" fill="10" visible="yes" active="yes"/>
 <layer number="43" name="vRestrict" color="2" fill="10" visible="no" active="yes"/>
@@
 <layer number="49" name="Reference" color="7" fill="1" visible="no" active="yes"/>
 <layer number="50" name="dxf" color="7" fill="1" visible="no" active="no"/>
-<layer number="51" name="tDocu" color="7" fill="1" visible="no" active="yes"/>
-<layer number="52" name="bDocu" color="7" fill="1" visible="no" active="yes"/>
+<layer number="51" name="tDocu" color="7" fill="1" visible="yes" active="yes"/>
+<layer number="52" name="bDocu" color="7" fill="1" visible="yes" active="yes"/>
 <layer number="53" name="tGND_GNDA" color="7" fill="1" visible="no" active="no"/>
 <layer number="54" name="bGND_GNDA" color="7" fill="1" visible="no" active="no"/>
@@
 <wire x1="10.9" y1="-23.77" x2="12.13" y2="-25" width="0" layer="20" curve="90"/>
 <wire x1="12.13" y1="-25" x2="45.195" y2="-25" width="0" layer="20"/>
-<text x="23.8184" y="-6.4804" size="1.27" layer="25" rot="R90" align="center">CLK</text>
-<text x="25.9266" y="-6.455" size="1.27" layer="25" rot="R90" align="center">DIO</text>
-<text x="28.9086" y="-5.5694" size="1.27" layer="25" rot="R180" align="center">TX</text>
-<text x="31.4448" y="-5.6964" size="1.27" layer="25" rot="R180" align="center">G</text>
+<text x="23.8184" y="-6.4804" size="1.27" layer="51" rot="R90" align="center">CLK</text>
+<text x="25.9266" y="-6.455" size="1.27" layer="51" rot="R90" align="center">DIO</text>
+<text x="28.9086" y="-5.5694" size="1.27" layer="51" rot="R180" align="center">TX</text>
+<text x="31.4448" y="-5.6964" size="1.27" layer="51" rot="R180" align="center">G</text>
 <wire x1="45.195" y1="-25" x2="47.1" y2="-23.095" width="0" layer="20" curve="90"/>
-<text x="21.3174" y="-6.6552" size="1.27" layer="25" rot="R270" align="center">3V3</text>
+<text x="21.3174" y="-6.6552" size="1.27" layer="51" rot="R270" align="center">3V3</text>
 <text x="10.0144" y="-0.1782" size="1.27" layer="25" rot="R270" align="center">GND</text>
 <text x="7.4744" y="0.8378" size="1.27" layer="25" rot="R270" align="center">HSHOE</text>
@@
 <text x="-5.6638" y="-23.5136" size="1.9304" layer="25" align="center">USER</text>
 <text x="18.5932" y="-23.3866" size="1.9304" layer="25" align="center">RESET</text>
-<text x="0.381" y="-20.32" size="2.1844" layer="25" align="center">ON</text>
-<text x="12.319" y="-20.32" size="2.1844" layer="25" align="center">OFF</text>
+<text x="0.635" y="-17.78" size="2.1844" layer="25" align="center">ON</text>
+<text x="11.811" y="-17.78" size="2.1844" layer="25" align="center">OFF</text>
 <rectangle x1="-4.064" y1="-17.907" x2="4.318" y2="-10.541" layer="16"/>
 <text x="32.639" y="-13.208" size="1.27" layer="25" rot="R90" align="center">PC</text>
 <text x="32.639" y="-15.875" size="1.27" layer="25" align="center">G</text>
-<text x="-6.35" y="-3.223" size="1.27" layer="25" rot="R180" align="center">S</text>
+<text x="-5.969" y="-3.096" size="1.27" layer="25" rot="R180" align="center">LS</text>
 <text x="-10.4744" y="-4.6478" size="1.27" layer="25" rot="R90" align="center">G</text>
 <text x="-14.5538" y="-3.1146" size="1.27" layer="25" align="center">V</text>
@@
 <attribute name="NAME" x="-13.335" y="-19.4945" size="0.8128" layer="25" rot="R180"/>
 </element>
-<element name="U$10" library="apricot" package="HOTSHOE_RAIL" value="HOTSHOE" x="14.102" y="14.688" smashed="yes" rot="MR0"/>
-<element name="U$15" library="apricot" package="HOTSHOE_RAIL" value="HOTSHOE" x="-1.455" y="14.688" smashed="yes" rot="MR0"/>
-<element name="U$2" library="apricot" package="SPRING_CONTACT" value="SPRING_CONTACT" x="6.3" y="10.3" smashed="yes" rot="MR0"/>
+<element name="U$10" library="apricot" package="HOTSHOE_RAIL_NOPASTE" value="HOTSHOE_NOPASTE" x="14.102" y="14.688" smashed="yes" rot="MR0"/>
+<element name="U$15" library="apricot" package="HOTSHOE_RAIL_NOPASTE" value="HOTSHOE_NOPASTE" x="-1.455" y="14.688" smashed="yes" rot="MR0"/>
+<element name="U$2" library="apricot" package="SPRING_CONTACT" value="SPRING_CONTACT" x="6.3" y="10.05" smashed="yes" rot="MR0"/>
 <element name="U$3" library="apricot" package="HOTSHOE_RAIL" value="HOTSHOE" x="-1.397" y="14.732" smashed="yes"/>
 <element name="U$4" library="apricot" package="HOTSHOE_RAIL" value="HOTSHOE" x="14.097" y="14.732" smashed="yes"/>
-<element name="U$5" library="apricot" package="HOTSHOE_RAIL" value="HOTSHOE" x="-1.397" y="3.048" smashed="yes" rot="MR0"/>
-<element name="U$9" library="apricot" package="HOTSHOE_RAIL" value="HOTSHOE" x="14.097" y="3.048" smashed="yes" rot="MR0"/>
+<element name="U$5" library="apricot" package="HOTSHOE_RAIL_NOPASTE" value="HOTSHOE_NOPASTE" x="-1.397" y="3.048" smashed="yes" rot="MR0"/>
+<element name="U$9" library="apricot" package="HOTSHOE_RAIL_NOPASTE" value="HOTSHOE_NOPASTE" x="14.097" y="3.048" smashed="yes" rot="MR0"/>
 <element name="U$14" library="apricot" package="HOTSHOE_RAIL" value="HOTSHOE" x="-1.397" y="3.048" smashed="yes"/>
 <element name="U$16" library="apricot" package="HOTSHOE_RAIL" value="HOTSHOE" x="14.097" y="3.048" smashed="yes"/>
@@
 <wire x1="6.35" y1="-3.048" x2="7.493" y2="-3.048" width="0.3048" layer="16"/>
 <wire x1="6.3" y1="-2.998" x2="6.35" y2="-3.048" width="0.3048" layer="16"/>
-<wire x1="6.3" y1="10.3" x2="6.3" y2="-2.998" width="0.3048" layer="16"/>
+<wire x1="6.3" y1="10.05" x2="6.3" y2="-2.998" width="0.3048" layer="16"/>
 <wire x1="7.493" y1="-3.048" x2="7.493" y2="-4.191" width="0.2032" layer="1"/>
 <wire x1="8.255" y1="-4.953" x2="17.007" y2="-4.953" width="0.2032" layer="1"/>
