File: pcb/pmm.sch (EAGLE design)
At the start: 39 parts, among them IC3 STM32F042F4, J1 AUDIO_JACK_3.5MM_PTH, J2 FFC3B07-05-T, SW3 324_SW, SW4 324_SW, U2 USBC_16P, U4 XC6206_DEV

Commit message: cleaning up pcb
Parts:
- added U$14, U$16, U$5, U$9: HOTSHOE, apricot:HOTSHOE
- C2, C23: value 2.2uF -> 1uF
- C3: value 1uF -> 2.2uF
- R4: value 2K -> 5.1K
Connections:
- net +3V3: now also C3.2
- net GND: now also U$14.P$1, U$16.P$1, U$5.P$1, U$9.P$1
- net N$3: no longer C3.2
Changed lines of the file:
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@@
 <part name="SW4" library="3pos_slide_switch_centered" deviceset="324_SW" device="" value="324_SW"/>
 <part name="LED1" library="adafruit" deviceset="LED" device="CHIP-LED0805"/>
-<part name="R4" library="SparkFun-Passives" deviceset="RESISTOR" device="0805-RES" value="2K"/>
+<part name="R4" library="SparkFun-Passives" deviceset="RESISTOR" device="0805-RES" value="5.1K"/>
 <part name="+3V2" library="supply1" library_urn="urn:adsk.eagle:library:371" deviceset="+3V3" device=""/>
 <part name="R5" library="joyAnalog" deviceset="RESISTOR" device="0805-RES" value="10K"/>
 <part name="GND10" library="supply1" deviceset="GND" device=""/>
 <part name="U4" library="3pos_slide_switch" deviceset="XC6206_DEV" device=""/>
-<part name="C2" library="clock" deviceset="CAP" device="0805" value="2.2uF"/>
+<part name="C2" library="clock" deviceset="CAP" device="0805" value="1uF"/>
 <part name="+3V3" library="supply1" library_urn="urn:adsk.eagle:library:371" deviceset="+3V3" device=""/>
 <part name="U$12" library="3pos_slide_switch_centered" deviceset="M2_SCREW_DEV" device=""/>
@@
 <part name="GND27" library="supply1" library_urn="urn:adsk.eagle:library:371" deviceset="GND" device=""/>
 <part name="C22" library="clock" deviceset="CAP" device="0805" value="2.2uF"/>
-<part name="C23" library="clock" deviceset="CAP" device="0805" value="2.2uF"/>
+<part name="C23" library="clock" deviceset="CAP" device="0805" value="1uF"/>
 <part name="GND28" library="supply1" library_urn="urn:adsk.eagle:library:371" deviceset="GND" device=""/>
 <part name="GND29" library="supply1" library_urn="urn:adsk.eagle:library:371" deviceset="GND" device=""/>
@@
 <part name="J1" library="SparkFun-Connectors" deviceset="AUDIO_JACK_3.5MM" device="_PTH"/>
 <part name="J2" library="FFC3B07-05-T" deviceset="FFC3B07-05-T" device=""/>
-<part name="GND3" library="supply1" deviceset="GND" device=""/>
 <part name="GND4" library="supply1" deviceset="GND" device=""/>
 <part name="U$6" library="adafruit_changed" deviceset="PINHD5" device=""/>
@@
 <part name="GND18" library="supply1" deviceset="GND" device=""/>
 <part name="GND19" library="supply1" deviceset="GND" device=""/>
-<part name="C3" library="clock" deviceset="CAP" device="0805" value="1uF"/>
+<part name="C3" library="clock" deviceset="CAP" device="0805" value="2.2uF"/>
 <part name="GND20" library="supply1" deviceset="GND" device=""/>
 <part name="JP2" library="adafruit_changed" deviceset="PINHD-1X3" device="CB"/>
@@
 <part name="GND2" library="supply1" deviceset="GND" device=""/>
 <part name="GND22" library="supply1" deviceset="GND" device=""/>
+<part name="U$5" library="apricot" deviceset="HOTSHOE" device=""/>
+<part name="U$9" library="apricot" deviceset="HOTSHOE" device=""/>
+<part name="GND25" library="supply1" deviceset="GND" device=""/>
+<part name="GND31" library="supply1" deviceset="GND" device=""/>
+<part name="U$14" library="apricot" deviceset="HOTSHOE" device=""/>
+<part name="U$16" library="apricot" deviceset="HOTSHOE" device=""/>
+<part name="GND34" library="supply1" deviceset="GND" device=""/>
+<part name="GND35" library="supply1" deviceset="GND" device=""/>
+<part name="+3V11" library="supply1" library_urn="urn:adsk.eagle:library:371" deviceset="+3V3" device=""/>
 </parts>
 <sheets>
@@
 <attribute name="VALUE" x="-5.08" y="53.34" size="1.778" layer="96"/>
 </instance>
-<instance part="GND3" gate="1" x="-106.68" y="-27.94" smashed="yes" rot="MR0">
-<attribute name="VALUE" x="-104.14" y="-30.48" size="1.778" layer="96" rot="MR0"/>
-</instance>
 <instance part="GND4" gate="1" x="-96.52" y="25.4" smashed="yes" rot="MR0">
 <attribute name="VALUE" x="-93.98" y="22.86" size="1.778" layer="96" rot="MR0"/>
@@
 <instance part="GND22" gate="1" x="-116.84" y="160.02" smashed="yes" rot="MR0">
 <attribute name="VALUE" x="-114.3" y="157.48" size="1.778" layer="96" rot="MR0"/>
+</instance>
+<instance part="U$5" gate="G$1" x="-93.98" y="205.74" smashed="yes"/>
+<instance part="U$9" gate="G$1" x="-93.98" y="185.42" smashed="yes"/>
+<instance part="GND25" gate="1" x="-109.22" y="182.88" smashed="yes" rot="MR0">
+<attribute name="VALUE" x="-106.68" y="180.34" size="1.778" layer="96" rot="MR0"/>
+</instance>
+<instance part="GND31" gate="1" x="-109.22" y="203.2" smashed="yes" rot="MR0">
+<attribute name="VALUE" x="-106.68" y="200.66" size="1.778" layer="96" rot="MR0"/>
+</instance>
+<instance part="U$14" gate="G$1" x="-167.64" y="203.2" smashed="yes"/>
+<instance part="U$16" gate="G$1" x="-167.64" y="182.88" smashed="yes"/>
+<instance part="GND34" gate="1" x="-182.88" y="180.34" smashed="yes" rot="MR0">
+<attribute name="VALUE" x="-180.34" y="177.8" size="1.778" layer="96" rot="MR0"/>
+</instance>
+<instance part="GND35" gate="1" x="-182.88" y="200.66" smashed="yes" rot="MR0">
+<attribute name="VALUE" x="-180.34" y="198.12" size="1.778" layer="96" rot="MR0"/>
+</instance>
+<instance part="+3V11" gate="G$1" x="360.68" y="35.56" smashed="yes" rot="MR0">
+<attribute name="VALUE" x="355.6" y="30.48" size="1.778" layer="96" rot="MR90"/>
 </instance>
 </instances>
@@
 <wire x1="-111.76" y1="142.24" x2="-116.84" y2="142.24" width="0.1524" layer="91"/>
 </segment>
+<segment>
+<pinref part="GND31" gate="1" pin="GND"/>
+<pinref part="U$5" gate="G$1" pin="P$1"/>
+<wire x1="-109.22" y1="205.74" x2="-104.14" y2="205.74" width="0.1524" layer="91"/>
+</segment>
+<segment>
+<pinref part="U$9" gate="G$1" pin="P$1"/>
+<pinref part="GND25" gate="1" pin="GND"/>
+<wire x1="-104.14" y1="185.42" x2="-109.22" y2="185.42" width="0.1524" layer="91"/>
+</segment>
+<segment>
+<pinref part="GND35" gate="1" pin="GND"/>
+<pinref part="U$14" gate="G$1" pin="P$1"/>
+<wire x1="-182.88" y1="203.2" x2="-177.8" y2="203.2" width="0.1524" layer="91"/>
+</segment>
+<segment>
+<pinref part="U$16" gate="G$1" pin="P$1"/>
+<pinref part="GND34" gate="1" pin="GND"/>
+<wire x1="-177.8" y1="182.88" x2="-182.88" y2="182.88" width="0.1524" layer="91"/>
+</segment>
 </net>
 <net name="+3V3" class="0">
@@
 <pinref part="+3V9" gate="G$1" pin="+3V3"/>
 <wire x1="-58.42" y1="63.5" x2="-68.58" y2="63.5" width="0.1524" layer="91"/>
+</segment>
+<segment>
+<pinref part="C3" gate="G$1" pin="2"/>
+<wire x1="360.68" y1="33.02" x2="360.68" y2="30.48" width="0.1524" layer="91"/>
+<pinref part="+3V11" gate="G$1" pin="+3V3"/>
 </segment>
 </net>
@@
 <pinref part="JP1" gate="A" pin="3"/>
 <wire x1="345.44" y1="33.02" x2="345.44" y2="15.24" width="0.1524" layer="91"/>
-<pinref part="C3" gate="G$1" pin="2"/>
-<wire x1="360.68" y1="33.02" x2="360.68" y2="30.48" width="0.1524" layer="91"/>
-<wire x1="345.44" y1="33.02" x2="360.68" y2="33.02" width="0.1524" layer="91"/>
-<junction x="345.44" y="33.02"/>
-</segment>
-</net>
+</segment>
+</net>

Commit message: cleaning up pcb
Parts:
- U$10, U$15, U$5, U$9: value HOTSHOE -> HOTSHOE_NOPASTE; device apricot:HOTSHOE -> apricot:HOTSHOE_NOPASTE
Changed lines of the file:
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@@
 <part name="R9" library="joyAnalog" deviceset="RESISTOR" device="0805-RES" value="270K"/>
 <part name="GND21" library="supply1" deviceset="GND" device=""/>
-<part name="U$10" library="apricot" deviceset="HOTSHOE" device=""/>
-<part name="U$15" library="apricot" deviceset="HOTSHOE" device=""/>
+<part name="U$10" library="apricot" deviceset="HOTSHOE_NOPASTE" device=""/>
+<part name="U$15" library="apricot" deviceset="HOTSHOE_NOPASTE" device=""/>
 <part name="GND23" library="supply1" deviceset="GND" device=""/>
 <part name="GND24" library="supply1" deviceset="GND" device=""/>
@@
 <part name="GND2" library="supply1" deviceset="GND" device=""/>
 <part name="GND22" library="supply1" deviceset="GND" device=""/>
-<part name="U$5" library="apricot" deviceset="HOTSHOE" device=""/>
-<part name="U$9" library="apricot" deviceset="HOTSHOE" device=""/>
+<part name="U$5" library="apricot" deviceset="HOTSHOE_NOPASTE" device=""/>
+<part name="U$9" library="apricot" deviceset="HOTSHOE_NOPASTE" device=""/>
 <part name="GND25" library="supply1" deviceset="GND" device=""/>
 <part name="GND31" library="supply1" deviceset="GND" device=""/>
@@
 <attribute name="VALUE" x="-25.4" y="53.34" size="1.778" layer="96" rot="MR0"/>
 </instance>
-<instance part="U$10" gate="G$1" x="-101.6" y="124.46" smashed="yes"/>
-<instance part="U$15" gate="G$1" x="-101.6" y="104.14" smashed="yes"/>
-<instance part="GND23" gate="1" x="-116.84" y="101.6" smashed="yes" rot="MR0">
-<attribute name="VALUE" x="-114.3" y="99.06" size="1.778" layer="96" rot="MR0"/>
-</instance>
-<instance part="GND24" gate="1" x="-116.84" y="121.92" smashed="yes" rot="MR0">
-<attribute name="VALUE" x="-114.3" y="119.38" size="1.778" layer="96" rot="MR0"/>
+<instance part="U$10" gate="G$1" x="-48.26" y="205.74" smashed="yes"/>
+<instance part="U$15" gate="G$1" x="-48.26" y="185.42" smashed="yes"/>
+<instance part="GND23" gate="1" x="-63.5" y="182.88" smashed="yes" rot="MR0">
+<attribute name="VALUE" x="-60.96" y="180.34" size="1.778" layer="96" rot="MR0"/>
+</instance>
+<instance part="GND24" gate="1" x="-63.5" y="203.2" smashed="yes" rot="MR0">
+<attribute name="VALUE" x="-60.96" y="200.66" size="1.778" layer="96" rot="MR0"/>
 </instance>
 <instance part="U$2" gate="G$1" x="-78.74" y="7.62" smashed="yes" rot="R180"/>
@@
 <pinref part="GND24" gate="1" pin="GND"/>
 <pinref part="U$10" gate="G$1" pin="P$1"/>
-<wire x1="-116.84" y1="124.46" x2="-111.76" y2="124.46" width="0.1524" layer="91"/>
+<wire x1="-63.5" y1="205.74" x2="-58.42" y2="205.74" width="0.1524" layer="91"/>
 </segment>
 <segment>
 <pinref part="U$15" gate="G$1" pin="P$1"/>
 <pinref part="GND23" gate="1" pin="GND"/>
-<wire x1="-111.76" y1="104.14" x2="-116.84" y2="104.14" width="0.1524" layer="91"/>
-</segment>
-<segment>
+<wire x1="-58.42" y1="185.42" x2="-63.5" y2="185.42" width="0.1524" layer="91"/>
+</segment>
+<segment>

Commit message: cleaning up pcb
Parts:
- added U$11, U$13: HOTSHOE_NOPASTE, apricot:HOTSHOE_NOPASTE
Connections:
- net GND: now also U$11.P$1, U$13.P$1
Changed lines of the file:
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@@
 <part name="GND35" library="supply1" deviceset="GND" device=""/>
 <part name="+3V11" library="supply1" library_urn="urn:adsk.eagle:library:371" deviceset="+3V3" device=""/>
+<part name="U$11" library="apricot" deviceset="HOTSHOE_NOPASTE" device=""/>
+<part name="GND3" library="supply1" deviceset="GND" device=""/>
+<part name="U$13" library="apricot" deviceset="HOTSHOE_NOPASTE" device=""/>
+<part name="GND32" library="supply1" deviceset="GND" device=""/>
 </parts>
 <sheets>
@@
 <instance part="+3V11" gate="G$1" x="360.68" y="35.56" smashed="yes" rot="MR0">
 <attribute name="VALUE" x="355.6" y="30.48" size="1.778" layer="96" rot="MR90"/>
+</instance>
+<instance part="U$11" gate="G$1" x="-48.26" y="223.52" smashed="yes"/>
+<instance part="GND3" gate="1" x="-63.5" y="220.98" smashed="yes" rot="MR0">
+<attribute name="VALUE" x="-60.96" y="218.44" size="1.778" layer="96" rot="MR0"/>
+</instance>
+<instance part="U$13" gate="G$1" x="-93.98" y="223.52" smashed="yes"/>
+<instance part="GND32" gate="1" x="-109.22" y="220.98" smashed="yes" rot="MR0">
+<attribute name="VALUE" x="-106.68" y="218.44" size="1.778" layer="96" rot="MR0"/>
 </instance>
 </instances>
@@
 <wire x1="-177.8" y1="182.88" x2="-182.88" y2="182.88" width="0.1524" layer="91"/>
 </segment>
+<segment>
+<pinref part="GND3" gate="1" pin="GND"/>
+<pinref part="U$11" gate="G$1" pin="P$1"/>
+<wire x1="-63.5" y1="223.52" x2="-58.42" y2="223.52" width="0.1524" layer="91"/>
+</segment>
+<segment>
+<pinref part="GND32" gate="1" pin="GND"/>
+<pinref part="U$13" gate="G$1" pin="P$1"/>
+<wire x1="-109.22" y1="223.52" x2="-104.14" y2="223.52" width="0.1524" layer="91"/>
+</segment>
 </net>
