File: pcb/rev2/pmm.sch (EAGLE design)
At the start: 45 parts, among them IC3 STM32F042F4, J1 AUDIO_JACK_3.5MM_PTH, J2 FFC3B07-05-T, SW4 324_SW, U2 USBC_16P, U4 XC6206_DEV

Commit message: working on improvments
Parts:
- added TP1, TP2, TP3: TPTP18R, testpad:TPTP18R
Connections:
- net +3V3: now also TP3.TP
- net GND: now also TP2.TP
- net LS_EXT: now also JP3.1
- net LS_INTERNAL: now also JP3.3
- net LS_MCU: now also TP1.TP
Other:
- moved on the sheet: R9
Changed lines of the file:
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@@
 <part name="R9" library="joyAnalog" deviceset="RESISTOR" device="0805-RES" value="270K"/>
 <part name="GND19" library="supply1" deviceset="GND" device=""/>
+<part name="TP1" library="testpad" library_urn="urn:adsk.eagle:library:385" deviceset="TP" device="TP18R" package3d_urn="urn:adsk.eagle:package:27981/1" value="TPTP18R"/>
+<part name="TP2" library="testpad" library_urn="urn:adsk.eagle:library:385" deviceset="TP" device="TP18R" package3d_urn="urn:adsk.eagle:package:27981/1" value="TPTP18R"/>
+<part name="TP3" library="testpad" library_urn="urn:adsk.eagle:library:385" deviceset="TP" device="TP18R" package3d_urn="urn:adsk.eagle:package:27981/1" value="TPTP18R"/>
+<part name="+3V9" library="supply1" library_urn="urn:adsk.eagle:library:371" deviceset="+3V3" device=""/>
+<part name="GND21" library="supply1" deviceset="GND" device=""/>
 </parts>
 <sheets>
@@
 <attribute name="VALUE" x="-167.64" y="101.6" size="1.778" layer="96" rot="MR90"/>
 </instance>
-<instance part="R9" gate="G$1" x="-147.32" y="15.24" smashed="yes" rot="MR270">
-<attribute name="NAME" x="-148.8186" y="16.51" size="1.778" layer="95" rot="MR270"/>
-<attribute name="VALUE" x="-151.638" y="19.05" size="1.778" layer="96" rot="MR270"/>
-</instance>
-<instance part="GND19" gate="1" x="-147.32" y="7.62" smashed="yes" rot="MR0">
-<attribute name="VALUE" x="-144.78" y="5.08" size="1.778" layer="96" rot="MR0"/>
+<instance part="R9" gate="G$1" x="-165.1" y="15.24" smashed="yes" rot="MR270">
+<attribute name="NAME" x="-166.5986" y="16.51" size="1.778" layer="95" rot="MR270"/>
+<attribute name="VALUE" x="-169.418" y="19.05" size="1.778" layer="96" rot="MR270"/>
+</instance>
+<instance part="GND19" gate="1" x="-165.1" y="7.62" smashed="yes" rot="MR0">
+<attribute name="VALUE" x="-162.56" y="5.08" size="1.778" layer="96" rot="MR0"/>
+</instance>
+<instance part="TP1" gate="G$1" x="-162.56" y="22.86" smashed="yes">
+<attribute name="NAME" x="-163.83" y="24.13" size="1.778" layer="95"/>
+<attribute name="TP_SIGNAL_NAME" x="-161.29" y="21.59" size="1.778" layer="97"/>
+</instance>
+<instance part="TP2" gate="G$1" x="-195.58" y="43.18" smashed="yes">
+<attribute name="NAME" x="-196.85" y="44.45" size="1.778" layer="95"/>
+<attribute name="TP_SIGNAL_NAME" x="-194.31" y="41.91" size="1.778" layer="97"/>
+</instance>
+<instance part="TP3" gate="G$1" x="-167.64" y="48.26" smashed="yes">
+<attribute name="NAME" x="-168.91" y="49.53" size="1.778" layer="95"/>
+<attribute name="TP_SIGNAL_NAME" x="-166.37" y="46.99" size="1.778" layer="97"/>
+</instance>
+<instance part="+3V9" gate="G$1" x="-162.56" y="48.26" smashed="yes" rot="MR0">
+<attribute name="VALUE" x="-160.02" y="43.18" size="1.778" layer="96" rot="MR90"/>
+</instance>
+<instance part="GND21" gate="1" x="-195.58" y="38.1" smashed="yes" rot="MR0">
+<attribute name="VALUE" x="-193.04" y="35.56" size="1.778" layer="96" rot="MR0"/>
 </instance>
 </instances>
@@
 <pinref part="GND19" gate="1" pin="GND"/>
 </segment>
+<segment>
+<pinref part="TP2" gate="G$1" pin="TP"/>
+<pinref part="GND21" gate="1" pin="GND"/>
+</segment>
 </net>
 <net name="+3V3" class="0">
@@
 <wire x1="-208.28" y1="104.14" x2="-215.9" y2="104.14" width="0.1524" layer="91"/>
 <pinref part="+3V12" gate="G$1" pin="+3V3"/>
+</segment>
+<segment>
+<pinref part="+3V9" gate="G$1" pin="+3V3"/>
+<pinref part="TP3" gate="G$1" pin="TP"/>
+<wire x1="-162.56" y1="45.72" x2="-167.64" y2="45.72" width="0.1524" layer="91"/>
 </segment>
 </net>
@@
 <label x="-198.12" y="71.12" size="1.778" layer="95"/>
 </segment>
+<segment>
+<pinref part="JP3" gate="A" pin="3"/>
+<wire x1="-129.54" y1="17.78" x2="-154.94" y2="17.78" width="0.1524" layer="91"/>
+<label x="-154.94" y="17.78" size="1.778" layer="95"/>
+</segment>
 </net>
 <net name="LS_EXT" class="0">
@@
 <label x="-48.26" y="68.58" size="1.778" layer="95"/>
 </segment>
+<segment>
+<pinref part="JP3" gate="A" pin="1"/>
+<wire x1="-129.54" y1="22.86" x2="-154.94" y2="22.86" width="0.1524" layer="91"/>
+<label x="-154.94" y="22.86" size="1.778" layer="95"/>
+</segment>
 </net>
 <net name="LS_MCU" class="0">
 <segment>
-<wire x1="-149.86" y1="20.32" x2="-147.32" y2="20.32" width="0.1524" layer="91"/>
-<label x="-147.32" y="20.32" size="1.778" layer="95"/>
+<wire x1="-167.64" y1="20.32" x2="-165.1" y2="20.32" width="0.1524" layer="91"/>
+<label x="-175.26" y="20.32" size="1.778" layer="95"/>
 <pinref part="JP3" gate="A" pin="2"/>
 <pinref part="R9" gate="G$1" pin="1"/>
-<wire x1="-147.32" y1="20.32" x2="-129.54" y2="20.32" width="0.1524" layer="91"/>
-<junction x="-147.32" y="20.32"/>
+<wire x1="-165.1" y1="20.32" x2="-162.56" y2="20.32" width="0.1524" layer="91"/>
+<junction x="-165.1" y="20.32"/>
+<pinref part="TP1" gate="G$1" pin="TP"/>
+<wire x1="-162.56" y1="20.32" x2="-129.54" y2="20.32" width="0.1524" layer="91"/>
+<junction x="-162.56" y="20.32"/>
 </segment>
 <segment>
@@
 will not be understood (or retained) with this version.
 </note>
+<note version="8.3" severity="warning">
+Since Version 8.3, EAGLE supports the association of 3D packages
+with devices in libraries, schematics, and board files. Those 3D
+packages will not be understood (or retained) with this version.
+</note>
 </compatibility>

Commit message: reset button
Parts:
- added SW3: 324_SW324_SWITCH_FOOT_HOLE, 3pos_slide_switch:324_SW324_SWITCH_FOOT_HOLE
Connections:
- removed net BUTTON1: IC3.NRST
- new net RESET: IC3.NRST, SW3.1, SW3.4
- net GND: now also SW3.2, SW3.3
Changed lines of the file:
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@@
 <layer number="154" name="FabDoc2" color="7" fill="1" visible="yes" active="yes"/>
 <layer number="155" name="FabDoc3" color="7" fill="1" visible="yes" active="yes"/>
+<layer number="156" name="gesam-Maß" color="7" fill="1" visible="no" active="yes"/>
+<layer number="157" name="FaceMchng" color="7" fill="1" visible="no" active="yes"/>
+<layer number="158" name="FaceMMeas" color="7" fill="1" visible="no" active="yes"/>
+<layer number="159" name="Geh-Bear2" color="7" fill="1" visible="no" active="yes"/>
+<layer number="160" name="O_Dim" color="7" fill="1" visible="yes" active="yes"/>
+<layer number="161" name="tomplace2" color="7" fill="1" visible="no" active="yes"/>
 <layer number="166" name="AntennaArea" color="7" fill="1" visible="yes" active="yes"/>
 <layer number="168" name="4mmHeightArea" color="7" fill="1" visible="yes" active="yes"/>
@@
 <layer number="250" name="Descript" color="3" fill="1" visible="no" active="no"/>
 <layer number="251" name="SMDround" color="12" fill="11" visible="no" active="no"/>
+<layer number="252" name="BR-BS" color="7" fill="1" visible="no" active="yes"/>
 <layer number="253" name="Extra" color="7" fill="1" visible="yes" active="yes"/>
 <layer number="254" name="cooling" color="7" fill="1" visible="yes" active="yes"/>
@@
 <part name="+3V9" library="supply1" library_urn="urn:adsk.eagle:library:371" deviceset="+3V3" device=""/>
 <part name="GND21" library="supply1" deviceset="GND" device=""/>
+<part name="SW3" library="3pos_slide_switch" deviceset="324_SW" device="324_SWITCH_FOOT_HOLE" value="324_SW324_SWITCH_FOOT_HOLE"/>
+<part name="GND33" library="supply1" deviceset="GND" device=""/>
 </parts>
 <sheets>
@@
 <instance part="GND21" gate="1" x="-195.58" y="38.1" smashed="yes" rot="MR0">
 <attribute name="VALUE" x="-193.04" y="35.56" size="1.778" layer="96" rot="MR0"/>
+</instance>
+<instance part="SW3" gate="G$1" x="147.32" y="60.96" smashed="yes"/>
+<instance part="GND33" gate="1" x="175.26" y="60.96" smashed="yes" rot="MR0">
+<attribute name="VALUE" x="177.8" y="58.42" size="1.778" layer="96" rot="MR0"/>
 </instance>
 </instances>
@@
 <pinref part="GND21" gate="1" pin="GND"/>
 </segment>
+<segment>
+<pinref part="SW3" gate="G$1" pin="3"/>
+<pinref part="SW3" gate="G$1" pin="2"/>
+<wire x1="162.56" y1="66.04" x2="132.08" y2="66.04" width="0.1524" layer="91"/>
+<pinref part="GND33" gate="1" pin="GND"/>
+<wire x1="162.56" y1="66.04" x2="175.26" y2="66.04" width="0.1524" layer="91"/>
+<wire x1="175.26" y1="66.04" x2="175.26" y2="63.5" width="0.1524" layer="91"/>
+<junction x="162.56" y="66.04"/>
+</segment>
 </net>
 <net name="+3V3" class="0">
@@
 </segment>
 </net>
-<net name="BUTTON1" class="0">
+<net name="RESET" class="0">
 <segment>
 <label x="40.64" y="33.02" size="1.778" layer="95"/>
 <pinref part="IC3" gate="G$1" pin="NRST"/>
-<wire x1="20.32" y1="33.02" x2="53.34" y2="33.02" width="0.1524" layer="91"/>
+<pinref part="SW3" gate="G$1" pin="1"/>
+<pinref part="SW3" gate="G$1" pin="4"/>
+<wire x1="132.08" y1="58.42" x2="162.56" y2="58.42" width="0.1524" layer="91"/>
+<wire x1="20.32" y1="33.02" x2="132.08" y2="33.02" width="0.1524" layer="91"/>
+<wire x1="132.08" y1="33.02" x2="132.08" y2="58.42" width="0.1524" layer="91"/>
+<junction x="132.08" y="58.42"/>
 </segment>
 </net>
