File: pcb/old/oldlight.sch (EAGLE design)
At the start: 6 parts, among them J3 FFC3B07-05-T

Commit message: photodiode
Parts:
- removed D1: BPW_34_S-Z, BPW_34_S-Z:BPW_34_S-Z
- removed U$1: LS_VERT, apricot:LS_VERT
- removed U$5: TLV2371DBV, texas-instruments:TLV2371DBV
- added JP1: (no value), adafruit_changed:PINHD-1X3CB
- added U1: TEMT6000, SparkFun:TEMT6000
- C1: value DNP -> 100nF
- R5: value 51K? -> 10K
Connections:
- removed net LS_SIGNAL: C1.1, J3.3, R5.1, U$1.B3, U$1.B4, U$1.T3, U$1.T4, U$5A.OUT
- removed net N$2: C1.2, D1.C, R5.2, U$5A.IN-
- new net S: J3.3, JP1.3, R5.2, U1.E1
- net +3V3: now also C1.2, JP1.1, U1.C1; no longer U$1.B1, U$1.B2, U$5SUPPLY.V+
- net GND: now also C1.1, JP1.2, R5.1; no longer D1.A, U$1.T1, U$1.T2, U$5A.IN+, U$5SUPPLY.V-
Other:
- moved on the sheet: C1, R5
